File: CurrentControl.sch (KiCad schematic (older format))
At the start: 7 parts

Commit message: Initial annotation.
Parts:
- gave numbers to parts that had none: 7
Changed lines of the file:
@@
 encoding utf-8
 Sheet 2 4
-Title ""
-Date ""
-Rev ""
-Comp ""
+Title "Current Control"
+Date "2016-06-12"
+Rev "-"
+Comp "J A"
 Comment1 ""
 Comment2 ""
@@
 $EndDescr
 $Comp
-L LMV358 U?
+L LMV358 U201
 U 1 1 575CD7DB
 P 5230 3610
-F 0 "U?" H 5180 3810 50  0000 L CNN
+F 0 "U201" H 5180 3810 50  0000 L CNN
 F 1 "LMV358" H 5180 3360 50  0000 L CNN
 F 2 "" H 5230 3610 50  0000 C CNN
@@
 $EndComp
 $Comp
-L R R?
+L R R203
 U 1 1 575CD7E3
 P 6750 4590
-F 0 "R?" V 6830 4590 50  0000 C CNN
+F 0 "R203" V 6830 4590 50  0000 C CNN
 F 1 ".1" V 6750 4590 50  0000 C CNN
 F 2 "" V 6680 4590 50  0000 C CNN
@@
 $EndComp
 $Comp
-L Q_NMOS_DGS Q?
+L Q_NMOS_DGS Q201
 U 1 1 575CD7F1
 P 6650 3610
-F 0 "Q?" H 6950 3660 50  0000 R CNN
+F 0 "Q201" H 6950 3660 50  0000 R CNN
 F 1 "BUK9575" H 7300 3560 50  0000 R CNN
 F 2 "" H 6850 3710 50  0000 C CNN
@@
 $EndComp
 $Comp
-L R R?
+L R R201
 U 1 1 575CD7F8
 P 4120 4100
-F 0 "R?" V 4200 4100 50  0000 C CNN
+F 0 "R201" V 4200 4100 50  0000 C CNN
 F 1 "R" V 4120 4100 50  0000 C CNN
 F 2 "" V 4050 4100 50  0000 C CNN
@@
 $EndComp
 $Comp
-L GND #PWR?
+L GND #PWR202
 U 1 1 575CD7FF
 P 5130 4020
-F 0 "#PWR?" H 5130 3770 50  0001 C CNN
+F 0 "#PWR202" H 5130 3770 50  0001 C CNN
 F 1 "GND" H 5130 3870 50  0000 C CNN
 F 2 "" H 5130 4020 50  0000 C CNN
@@
 $EndComp
 $Comp
-L POT-RESCUE-CSOS RV?
+L POT-RESCUE-CSOS RV201
 U 1 1 575CD805
 P 4120 3480
-F 0 "RV?" H 4120 3380 50  0000 C CNN
+F 0 "RV201" H 4120 3380 50  0000 C CNN
 F 1 "POT" H 4120 3480 50  0000 C CNN
 F 2 "" H 4120 3480 50  0000 C CNN
@@
 	4700 4240 6750 4240
 $Comp
-L C C?
+L C C201
 U 1 1 575CD820
 P 4780 3060
-F 0 "C?" H 4805 3160 50  0000 L CNN
+F 0 "C201" H 4805 3160 50  0000 L CNN
 F 1 "C" H 4805 2960 50  0000 L CNN
 F 2 "" H 4818 2910 50  0000 C CNN
@@
 $EndComp
 $Comp
-L GND #PWR?
+L GND #PWR201
 U 1 1 575CD827
 P 4780 3250
-F 0 "#PWR?" H 4780 3000 50  0001 C CNN
+F 0 "#PWR201" H 4780 3000 50  0001 C CNN
 F 1 "GND" H 4780 3100 50  0000 C CNN
 F 2 "" H 4780 3250 50  0000 C CNN
@@
 Connection ~ 4780 2830
 $Comp
-L R R?
+L R R202
 U 1 1 575D8253
 P 5970 3610
-F 0 "R?" V 6050 3610 50  0000 C CNN
+F 0 "R202" V 6050 3610 50  0000 C CNN
 F 1 "1K" V 5970 3610 50  0000 C CNN
 F 2 "" V 5900 3610 50  0000 C CNN

Commit message: Initial component association and global spread in layout.
Parts:
- C201: footprint (none) -> Capacitors_SMD:C_0805_HandSoldering
- Q201: footprint (none) -> TO_SOT_Packages_THT:TO-220_Neutral123_Vertical
- R201, R202: footprint (none) -> Resistors_SMD:R_0805_HandSoldering
- R203: footprint (none) -> Resistors_ThroughHole:Resistor_Horizontal_RM15mm
- RV201: footprint (none) -> Potentiometers:Potentiometer_WirePads_largePads
- U201: footprint (none) -> SMD_Packages:SOIC-8-N; MPN (none) -> LMV358IDT
Changed lines of the file:
@@
 F 0 "U201" H 5180 3810 50  0000 L CNN
 F 1 "LMV358" H 5180 3360 50  0000 L CNN
-F 2 "" H 5230 3610 50  0000 C CNN
-F 3 "" H 5230 3610 50  0000 C CNN
+F 2 "SMD_Packages:SOIC-8-N" H 5230 3610 50  0001 C CNN
+F 3 "http://www.st.com/content/ccc/resource/technical/document/datasheet/b9/d8/3b/8f/a1/8f/46/01/CD00079372.pdf/files/CD00079372.pdf/jcr:content/translations/en.CD00079372.pdf" H 5230 3610 50  0001 C CNN
+F 4 "LMV358IDT" H 5230 3610 60  0001 C CNN "MPN"
 	1    5230 3610
 	1    0    0    -1
@@
 F 0 "R203" V 6830 4590 50  0000 C CNN
 F 1 ".1" V 6750 4590 50  0000 C CNN
-F 2 "" V 6680 4590 50  0000 C CNN
+F 2 "Resistors_ThroughHole:Resistor_Horizontal_RM15mm" V 6680 4590 50  0001 C CNN
 F 3 "" H 6750 4590 50  0000 C CNN
 F 4 "AC01000001007JA100" V 6750 4590 60  0001 C CNN "MPN"
@@
 F 0 "Q201" H 6950 3660 50  0000 R CNN
 F 1 "BUK9575" H 7300 3560 50  0000 R CNN
-F 2 "" H 6850 3710 50  0000 C CNN
+F 2 "TO_SOT_Packages_THT:TO-220_Neutral123_Vertical" H 6850 3710 50  0001 C CNN
 F 3 "" H 6650 3610 50  0000 C CNN
 F 4 "BUK9575-100A,127 " H 6650 3610 60  0001 C CNN "MPN"
@@
 F 0 "R201" V 4200 4100 50  0000 C CNN
 F 1 "R" V 4120 4100 50  0000 C CNN
-F 2 "" V 4050 4100 50  0000 C CNN
+F 2 "Resistors_SMD:R_0805_HandSoldering" V 4050 4100 50  0001 C CNN
 F 3 "" H 4120 4100 50  0000 C CNN
 	1    4120 4100
@@
 $EndComp
 $Comp
-L GND #PWR202
+L GND #PWR03
 U 1 1 575CD7FF
 P 5130 4020
-F 0 "#PWR202" H 5130 3770 50  0001 C CNN
+F 0 "#PWR03" H 5130 3770 50  0001 C CNN
 F 1 "GND" H 5130 3870 50  0000 C CNN
 F 2 "" H 5130 4020 50  0000 C CNN
@@
 F 0 "RV201" H 4120 3380 50  0000 C CNN
 F 1 "POT" H 4120 3480 50  0000 C CNN
-F 2 "" H 4120 3480 50  0000 C CNN
+F 2 "Potentiometers:Potentiometer_WirePads_largePads" H 4120 3480 50  0001 C CNN
 F 3 "" H 4120 3480 50  0000 C CNN
 	1    4120 3480
@@
 F 0 "C201" H 4805 3160 50  0000 L CNN
 F 1 "C" H 4805 2960 50  0000 L CNN
-F 2 "" H 4818 2910 50  0000 C CNN
+F 2 "Capacitors_SMD:C_0805_HandSoldering" H 4818 2910 50  0001 C CNN
 F 3 "" H 4780 3060 50  0000 C CNN
 	1    4780 3060
@@
 $EndComp
 $Comp
-L GND #PWR201
+L GND #PWR04
 U 1 1 575CD827
 P 4780 3250
-F 0 "#PWR201" H 4780 3000 50  0001 C CNN
+F 0 "#PWR04" H 4780 3000 50  0001 C CNN
 F 1 "GND" H 4780 3100 50  0000 C CNN
 F 2 "" H 4780 3250 50  0000 C CNN
@@
 F 0 "R202" V 6050 3610 50  0000 C CNN
 F 1 "1K" V 5970 3610 50  0000 C CNN
-F 2 "" V 5900 3610 50  0000 C CNN
+F 2 "Resistors_SMD:R_0805_HandSoldering" V 5900 3610 50  0001 C CNN
 F 3 "" H 5970 3610 50  0000 C CNN
 	1    5970 3610

Commit message: Creating heatsink footprint and adding to schematic and layout.
Parts:
- added P201: CONN_01X01, CSOS:FA-T220-38E, symbol CONN_01X01
Changed lines of the file:
@@
 Text HLabel 7160 5020 2    60   Input ~ 0
 Current_Sink-
+$Comp
+L CONN_01X01 P201
+U 1 1 575F34AB
+P 8290 3650
+F 0 "P201" H 8290 3750 50  0000 C CNN
+F 1 "CONN_01X01" V 8390 3650 50  0000 C CNN
+F 2 "CSOS:FA-T220-38E" H 8290 3650 50  0001 C CNN
+F 3 "" H 8290 3650 50  0000 C CNN
+	1    8290 3650
+	1    0    0    -1
+$EndComp
 $EndSCHEMATC

Commit message: Built potentiometer and added to layout.
Parts:
- RV201: footprint Potentiometers:Potentiometer_WirePads_largePads -> CSOS:P090L-02F25BR10K
Changed lines of the file:
@@
 F 0 "RV201" H 4120 3380 50  0000 C CNN
 F 1 "POT" H 4120 3480 50  0000 C CNN
-F 2 "Potentiometers:Potentiometer_WirePads_largePads" H 4120 3480 50  0001 C CNN
+F 2 "CSOS:P090L-02F25BR10K" H 4120 3480 50  0001 C CNN
 F 3 "" H 4120 3480 50  0000 C CNN
 	1    4120 3480

Commit message: Fixing voltage dividers and adding values.
Parts:
- R201: value R -> 68K
- RV201: value POT -> 10K
Connections:
- net 2.7V: now also R201.1; no longer RV201.2
- net Current_Sink-: now also RV201.2; no longer R201.2
- net at RV201.1: now also R201.2, U201.3 (+)
- now unconnected: RV201.3
Other:
- moved on the sheet: R201, RV201
Changed lines of the file:
@@
 L R R201
 U 1 1 575CD7F8
-P 4120 4100
-F 0 "R201" V 4200 4100 50  0000 C CNN
-F 1 "R" V 4120 4100 50  0000 C CNN
-F 2 "Resistors_SMD:R_0805_HandSoldering" V 4050 4100 50  0001 C CNN
-F 3 "" H 4120 4100 50  0000 C CNN
-	1    4120 4100
+P 4120 3580
+F 0 "R201" V 4200 3580 50  0000 C CNN
+F 1 "68K" V 4120 3580 50  0000 C CNN
+F 2 "Resistors_SMD:R_0805_HandSoldering" V 4050 3580 50  0001 C CNN
+F 3 "" H 4120 3580 50  0000 C CNN
+	1    4120 3580
 	1    0    0    -1
 $EndComp
@@
 L POT-RESCUE-CSOS RV201
 U 1 1 575CD805
-P 4120 3480
-F 0 "RV201" H 4120 3380 50  0000 C CNN
-F 1 "POT" H 4120 3480 50  0000 C CNN
-F 2 "CSOS:P090L-02F25BR10K" H 4120 3480 50  0001 C CNN
-F 3 "" H 4120 3480 50  0000 C CNN
-	1    4120 3480
+P 3970 4250
+F 0 "RV201" H 3970 4150 50  0000 C CNN
+F 1 "10K" H 3970 4250 50  0000 C CNN
+F 2 "CSOS:P090L-02F25BR10K" H 3970 4250 50  0001 C CNN
+F 3 "" H 3970 4250 50  0000 C CNN
+	1    3970 4250
 	0    1    1    0
 $EndComp
@@
 	6750 3810 6750 4440
 Wire Wire Line
-	4270 1770 4270 3480
+	4270 1770 4270 3200
 Connection ~ 6750 4860
 Wire Wire Line
@@
 	1    0    0    -1
 $EndComp
+Wire Wire Line
+	4270 3200 4120 3200
+Wire Wire Line
+	4120 3200 4120 3430
+Wire Wire Line
+	4120 3950 3970 3950
+Wire Wire Line
+	3970 3950 3970 4000
 $EndSCHEMATC

Commit message: Fixing FET.
Parts:
- removed Q201: BUK9575, TO_SOT_Packages_THT:TO-220_Neutral123_Vertical, symbol Q_NMOS_DGS
- added Q201: Q_NMOS_GDS, TO_SOT_Packages_THT:TO-220_Neutral123_Vertical, symbol Q_NMOS_GDS
Connections:
- net Current_Sink+: now also Q201.2 (D)
- net FET_Gate: now also Q201.1 (G)
- net at R203.1, U201.2 (-): now also Q201.3 (S)
Changed lines of the file:
@@
-$EndComp
-$Comp
-L Q_NMOS_DGS Q201
-U 1 1 575CD7F1
-P 6650 3610
-F 0 "Q201" H 6950 3660 50  0000 R CNN
-F 1 "BUK9575" H 7300 3560 50  0000 R CNN
-F 2 "TO_SOT_Packages_THT:TO-220_Neutral123_Vertical" H 6850 3710 50  0001 C CNN
-F 3 "" H 6650 3610 50  0000 C CNN
-F 4 "BUK9575-100A,127 " H 6650 3610 60  0001 C CNN "MPN"
-	1    6650 3610
-	1    0    0    -1
 $EndComp
 $Comp
@@
 Wire Wire Line
 	3970 3950 3970 4000
+$Comp
+L Q_NMOS_GDS Q201
+U 1 1 5761F503
+P 6650 3610
+F 0 "Q201" H 6950 3660 50  0000 R CNN
+F 1 "Q_NMOS_GDS" H 7300 3560 50  0000 R CNN
+F 2 "TO_SOT_Packages_THT:TO-220_Neutral123_Vertical" H 6850 3710 50  0001 C CNN
+F 3 "" H 6650 3610 50  0000 C CNN
+F 4 "BUK9575-100A,127" H 6650 3610 60  0001 C CNN "MPN"
+	1    6650 3610
+	1    0    0    -1
+$EndComp
 $EndSCHEMATC

Commit message: Layout connected.
Connections:
- net at R202.2: now also U201.7; no longer U201.1
- net at Q201.3 (S), R203.1: now also U201.6 (-); no longer U201.2 (-)
- net at R201.2, RV201.1: now also U201.5 (+); no longer U201.3 (+)
Changed lines of the file:
@@
 $Comp
 L LMV358 U201
-U 1 1 575CD7DB
+U 2 1 575CD7DB
 P 5230 3610
 F 0 "U201" H 5180 3810 50  0000 L CNN
@@
 F 3 "http://www.st.com/content/ccc/resource/technical/document/datasheet/b9/d8/3b/8f/a1/8f/46/01/CD00079372.pdf/files/CD00079372.pdf/jcr:content/translations/en.CD00079372.pdf" H 5230 3610 50  0001 C CNN
 F 4 "LMV358IDT" H 5230 3610 60  0001 C CNN "MPN"
-	1    5230 3610
+	2    5230 3610
 	1    0    0    -1
 $EndComp
