File: CurrentControl.sch (KiCad schematic (older format))
At the start: 8 parts, among them P201 CONN_01X01, Q201 Q_NMOS_GDS, U201 LMV358

Commit message: Finalizing MPNs and passive values for BOM generation and ordering parts.
Parts:
- C201: value C -> .1; MPN (none) -> 08055C104KAT2A
- P201: MPN (none) -> FA-T220-38E
- Q201: MPN BUK9575-100A,127 -> PHP23NQ11T,127
- RV201: MPN (none) -> P090L-02F25BR10K
Changed lines of the file:
@@
 Date "2016-06-12"
 Rev "-"
-Comp "J A"
+Comp "Joseph Allan"
 Comment1 ""
 Comment2 ""
@@
 F 2 "CSOS:P090L-02F25BR10K" H 3970 4250 50  0001 C CNN
 F 3 "" H 3970 4250 50  0000 C CNN
+F 4 "P090L-02F25BR10K" H 3970 4250 60  0001 C CNN "MPN"
 	1    3970 4250
 	0    1    1    0
@@
 P 4780 3060
 F 0 "C201" H 4805 3160 50  0000 L CNN
-F 1 "C" H 4805 2960 50  0000 L CNN
+F 1 ".1" H 4805 2960 50  0000 L CNN
 F 2 "Capacitors_SMD:C_0805_HandSoldering" H 4818 2910 50  0001 C CNN
 F 3 "" H 4780 3060 50  0000 C CNN
+F 4 "08055C104KAT2A" H 4780 3060 60  0001 C CNN "MPN"
 	1    4780 3060
 	1    0    0    -1
@@
 F 2 "CSOS:FA-T220-38E" H 8290 3650 50  0001 C CNN
 F 3 "http://www.ohmite.com/cat/sink_f_r.pdf" H 8290 3650 50  0001 C CNN
+F 4 "FA-T220-38E" H 8290 3650 60  0001 C CNN "MPN"
 	1    8290 3650
 	1    0    0    -1
@@
 F 1 "Q_NMOS_GDS" H 7300 3560 50  0000 R CNN
 F 2 "TO_SOT_Packages_THT:TO-220_Neutral123_Vertical" H 6850 3710 50  0001 C CNN
-F 3 "" H 6650 3610 50  0000 C CNN
-F 4 "BUK9575-100A,127" H 6650 3610 60  0001 C CNN "MPN"
+F 3 "http://www.nxp.com/documents/data_sheet/PHP23NQ11T.pdf" H 6650 3610 50  0001 C CNN
+F 4 "PHP23NQ11T,127" H 6650 3610 60  0001 C CNN "MPN"
 	1    6650 3610
 	1    0    0    -1

Commit message: Updating FET MPN.
Parts:
- Q201: MPN PHP23NQ11T,127 -> IRL540NPBF
Changed lines of the file:
@@
 F 1 "Q_NMOS_GDS" H 7300 3560 50  0000 R CNN
 F 2 "TO_SOT_Packages_THT:TO-220_Neutral123_Vertical" H 6850 3710 50  0001 C CNN
-F 3 "http://www.nxp.com/documents/data_sheet/PHP23NQ11T.pdf" H 6650 3610 50  0001 C CNN
-F 4 "PHP23NQ11T,127" H 6650 3610 60  0001 C CNN "MPN"
+F 3 "" H 6650 3610 50  0001 C CNN
+F 4 "IRL540NPBF " H 6650 3610 60  0001 C CNN "MPN"
 	1    6650 3610
 	1    0    0    -1
