File: CSOS.sch (KiCad schematic (older format))
At the start: 3 parts, among them P1 CONN_01X02

Commit message: Initial annotation.
Parts:
- gave numbers to parts that had none: 2
- renumbered P1 to P103
Changed lines of the file:
@@
 encoding utf-8
 Sheet 1 4
-Title ""
-Date ""
-Rev ""
-Comp ""
+Title "Current Sink"
+Date "2016-06-12"
+Rev "-"
+Comp "J A"
 Comment1 ""
 Comment2 ""
@@
 $EndDescr
 $Comp
-L CONN_01X02 P1
+L CONN_01X02 P103
 U 1 1 5747A1AB
 P 7450 2280
-F 0 "P1" H 7450 2430 50  0000 C CNN
+F 0 "P103" H 7450 2430 50  0000 C CNN
 F 1 "CONN_01X02" V 7550 2280 50  0000 C CNN
 F 2 "" H 7450 2280 50  0000 C CNN
@@
 $EndComp
 Wire Wire Line
-	7250 2330 7250 4620
-Wire Wire Line
-	7250 4620 7250 5910
+	7250 2330 7250 5910
 Wire Wire Line
 	7080 2230 7250 2230
 $Comp
-L CONN_01X03 P?
+L CONN_01X03 P102
 U 1 1 574C18ED
 P 6980 1410
-F 0 "P?" H 6980 1610 50  0000 C CNN
+F 0 "P102" H 6980 1610 50  0000 C CNN
 F 1 "CONN_01X03" V 7080 1410 50  0000 C CNN
 F 2 "" H 6980 1410 50  0000 C CNN
@@
 	6980 1610 6980 2810
 Wire Wire Line
-	6880 1610 6880 1730
+	6880 1730 6880 1610
 Wire Wire Line
-	6880 1730 6530 1730
+	3910 1730 6880 1730
 $Comp
-L CONN_01X02 P?
+L CONN_01X02 P101
 U 1 1 574C4DEE
 P 3710 1780
-F 0 "P?" H 3710 1930 50  0000 C CNN
+F 0 "P101" H 3710 1930 50  0000 C CNN
 F 1 "CONN_01X02" V 3810 1780 50  0000 C CNN
 F 2 "" H 3710 1780 50  0000 C CNN
@@
 	-1   0    0    -1
 $EndComp
-Wire Wire Line
-	6530 1730 6530 1730
-Wire Wire Line
-	6530 1730 3910 1730
 $Comp
-L GND #PWR?
+L GND #PWR101
 U 1 1 574C54DB
 P 4150 1930
-F 0 "#PWR?" H 4150 1680 50  0001 C CNN
+F 0 "#PWR101" H 4150 1680 50  0001 C CNN
 F 1 "GND" H 4150 1780 50  0000 C CNN
 F 2 "" H 4150 1930 50  0000 C CNN
@@
 $EndSheet
 Wire Wire Line
-	7080 1610 7080 2230
-Wire Wire Line
-	7080 2230 7080 4320
-Wire Wire Line
-	7080 4320 7080 5640
+	7080 1610 7080 5640
 Wire Wire Line
 	7080 4320 6380 4320
@@
 	4690 4750 5010 4750
 $Comp
-L GND #PWR?
+L GND #PWR102
 U 1 1 575E35B8
 P 7250 5910
-F 0 "#PWR?" H 7250 5660 50  0001 C CNN
+F 0 "#PWR102" H 7250 5660 50  0001 C CNN
 F 1 "GND" H 7250 5760 50  0000 C CNN
 F 2 "" H 7250 5910 50  0000 C CNN

Commit message: Initial component association and global spread in layout.
Parts:
- P101, P103: footprint (none) -> Pin_Headers:Pin_Header_Angled_1x02
- P102: footprint (none) -> Pin_Headers:Pin_Header_Angled_1x03
Changed lines of the file:
@@
 F 0 "P103" H 7450 2430 50  0000 C CNN
 F 1 "CONN_01X02" V 7550 2280 50  0000 C CNN
-F 2 "" H 7450 2280 50  0000 C CNN
+F 2 "Pin_Headers:Pin_Header_Angled_1x02" H 7450 2280 50  0001 C CNN
 F 3 "" H 7450 2280 50  0000 C CNN
 	1    7450 2280
@@
 F 0 "P102" H 6980 1610 50  0000 C CNN
 F 1 "CONN_01X03" V 7080 1410 50  0000 C CNN
-F 2 "" H 6980 1410 50  0000 C CNN
+F 2 "Pin_Headers:Pin_Header_Angled_1x03" H 6980 1410 50  0001 C CNN
 F 3 "" H 6980 1410 50  0000 C CNN
 	1    6980 1410
@@
 F 0 "P101" H 3710 1930 50  0000 C CNN
 F 1 "CONN_01X02" V 3810 1780 50  0000 C CNN
-F 2 "" H 3710 1780 50  0000 C CNN
+F 2 "Pin_Headers:Pin_Header_Angled_1x02" H 3710 1780 50  0001 C CNN
 F 3 "" H 3710 1780 50  0000 C CNN
 	1    3710 1780
@@
 $EndComp
 $Comp
-L GND #PWR101
+L GND #PWR01
 U 1 1 574C54DB
 P 4150 1930
-F 0 "#PWR101" H 4150 1680 50  0001 C CNN
+F 0 "#PWR01" H 4150 1680 50  0001 C CNN
 F 1 "GND" H 4150 1780 50  0000 C CNN
 F 2 "" H 4150 1930 50  0000 C CNN
@@
 	4690 4750 5010 4750
 $Comp
-L GND #PWR102
+L GND #PWR02
 U 1 1 575E35B8
 P 7250 5910
-F 0 "#PWR102" H 7250 5660 50  0001 C CNN
+F 0 "#PWR02" H 7250 5660 50  0001 C CNN
 F 1 "GND" H 7250 5760 50  0000 C CNN
 F 2 "" H 7250 5910 50  0000 C CNN

Commit message: Built 200 mil pitch terminal block. Updated pcb layout with new footprints.
Parts:
- P101, P103: footprint Pin_Headers:Pin_Header_Angled_1x02 -> CSOS:Terminal_Block_200_mil
- P102: footprint Pin_Headers:Pin_Header_Angled_1x03 -> Pin_Headers:Pin_Header_Straight_1x03
Changed lines of the file:
@@
 F 0 "P103" H 7450 2430 50  0000 C CNN
 F 1 "CONN_01X02" V 7550 2280 50  0000 C CNN
-F 2 "Pin_Headers:Pin_Header_Angled_1x02" H 7450 2280 50  0001 C CNN
+F 2 "CSOS:Terminal_Block_200_mil" H 7450 2280 50  0001 C CNN
 F 3 "" H 7450 2280 50  0000 C CNN
 	1    7450 2280
@@
 F 0 "P102" H 6980 1610 50  0000 C CNN
 F 1 "CONN_01X03" V 7080 1410 50  0000 C CNN
-F 2 "Pin_Headers:Pin_Header_Angled_1x03" H 6980 1410 50  0001 C CNN
+F 2 "Pin_Headers:Pin_Header_Straight_1x03" H 6980 1410 50  0001 C CNN
 F 3 "" H 6980 1410 50  0000 C CNN
 	1    6980 1410
@@
 F 0 "P101" H 3710 1930 50  0000 C CNN
 F 1 "CONN_01X02" V 3810 1780 50  0000 C CNN
-F 2 "Pin_Headers:Pin_Header_Angled_1x02" H 3710 1780 50  0001 C CNN
+F 2 "CSOS:Terminal_Block_200_mil" H 3710 1780 50  0001 C CNN
 F 3 "" H 3710 1780 50  0000 C CNN
 	1    3710 1780

Commit message: Finalizing MPNs and passive values for BOM generation and ordering parts.
Parts:
- P101, P103: MPN (none) -> OSTTC022162
- P102: MPN (none) -> M20-9990346
Changed lines of the file:
@@
 Date "2016-06-12"
 Rev "-"
-Comp "J A"
+Comp "Joseph Allan"
 Comment1 ""
 Comment2 ""
@@
 F 2 "CSOS:Terminal_Block_200_mil" H 7450 2280 50  0001 C CNN
 F 3 "" H 7450 2280 50  0000 C CNN
+F 4 "OSTTC022162" H 7450 2280 60  0001 C CNN "MPN"
 	1    7450 2280
 	1    0    0    -1
@@
 F 2 "Pin_Headers:Pin_Header_Straight_1x03" H 6980 1410 50  0001 C CNN
 F 3 "" H 6980 1410 50  0000 C CNN
+F 4 "M20-9990346" H 6980 1410 60  0001 C CNN "MPN"
 	1    6980 1410
 	0    -1   -1   0
@@
 F 2 "CSOS:Terminal_Block_200_mil" H 3710 1780 50  0001 C CNN
 F 3 "" H 3710 1780 50  0000 C CNN
+F 4 "OSTTC022162" H 3710 1780 60  0001 C CNN "MPN"
 	1    3710 1780
 	-1   0    0    -1
