File: PowerRegulation.sch (KiCad schematic (older format))
At the start: 6 parts

Commit message: Initial annotation.
Parts:
- gave numbers to parts that had none: 6
Changed lines of the file:
@@
 Sheet 4 4
 Title ""
-Date ""
-Rev ""
-Comp ""
+Date "2016-06-12"
+Rev "-"
+Comp "J A"
 Comment1 ""
 Comment2 ""
@@
 $EndDescr
 $Comp
-L GND #PWR?
+L GND #PWR401
 U 1 1 575DAECE
 P 5280 4310
-F 0 "#PWR?" H 5280 4060 50  0001 C CNN
+F 0 "#PWR401" H 5280 4060 50  0001 C CNN
 F 1 "GND" H 5280 4160 50  0000 C CNN
 F 2 "" H 5280 4310 50  0000 C CNN
@@
 $EndComp
 $Comp
-L C C?
+L C C402
 U 1 1 575DAED4
 P 6150 3820
-F 0 "C?" H 6175 3920 50  0000 L CNN
+F 0 "C402" H 6175 3920 50  0000 L CNN
 F 1 "C" H 6175 3720 50  0000 L CNN
 F 2 "" H 6188 3670 50  0000 C CNN
@@
 $EndComp
 $Comp
-L C C?
+L C C401
 U 1 1 575DAEDB
 P 4430 3720
-F 0 "C?" H 4455 3820 50  0000 L CNN
+F 0 "C401" H 4455 3820 50  0000 L CNN
 F 1 "C" H 4455 3620 50  0000 L CNN
 F 2 "" H 4468 3570 50  0000 C CNN
@@
 $EndComp
 $Comp
-L R R?
+L R R401
 U 1 1 575DAEE2
 P 4660 3690
-F 0 "R?" V 4740 3690 50  0000 C CNN
+F 0 "R401" V 4740 3690 50  0000 C CNN
 F 1 "0" V 4660 3690 50  0000 C CNN
 F 2 "" V 4590 3690 50  0000 C CNN
@@
 	5280 4280 5280 4310
 $Comp
-L LM2931D-R U?
+L LM2931D-R U401
 U 1 1 575DAF03
 P 5220 3280
-F 0 "U?" H 5490 3070 50  0000 C CNN
+F 0 "U401" H 5490 3070 50  0000 C CNN
 F 1 "LM2931D-R" H 5240 3630 50  0000 C CNN
 F 2 "" H 5220 3280 50  0000 C CNN
@@
 $EndComp
 $Comp
-L R R?
+L R R402
 U 1 1 575DAF0A
 P 5830 3340
-F 0 "R?" V 5910 3340 50  0000 C CNN
+F 0 "R402" V 5910 3340 50  0000 C CNN
 F 1 "27K" V 5830 3340 50  0000 C CNN
 F 2 "" V 5760 3340 50  0000 C CNN
@@
 $EndComp
 $Comp
-L R R?
+L R R403
 U 1 1 575DAF11
 P 5830 3720
-F 0 "R?" V 5910 3720 50  0000 C CNN
+F 0 "R403" V 5910 3720 50  0000 C CNN
 F 1 "21.6K" V 5830 3720 50  0000 C CNN
 F 2 "" V 5760 3720 50  0000 C CNN

Commit message: Initial component association and global spread in layout.
Parts:
- C401, C402: footprint (none) -> Capacitors_SMD:C_0805_HandSoldering
- R401, R402, R403: footprint (none) -> Resistors_SMD:R_0805_HandSoldering
- U401: footprint (none) -> SMD_Packages:SOIC-8-N
Changed lines of the file:
@@
 $EndDescr
 $Comp
-L GND #PWR401
+L GND #PWR07
 U 1 1 575DAECE
 P 5280 4310
-F 0 "#PWR401" H 5280 4060 50  0001 C CNN
+F 0 "#PWR07" H 5280 4060 50  0001 C CNN
 F 1 "GND" H 5280 4160 50  0000 C CNN
 F 2 "" H 5280 4310 50  0000 C CNN
@@
 F 0 "C402" H 6175 3920 50  0000 L CNN
 F 1 "C" H 6175 3720 50  0000 L CNN
-F 2 "" H 6188 3670 50  0000 C CNN
+F 2 "Capacitors_SMD:C_0805_HandSoldering" H 6188 3670 50  0001 C CNN
 F 3 "" H 6150 3820 50  0000 C CNN
 	1    6150 3820
@@
 F 0 "C401" H 4455 3820 50  0000 L CNN
 F 1 "C" H 4455 3620 50  0000 L CNN
-F 2 "" H 4468 3570 50  0000 C CNN
+F 2 "Capacitors_SMD:C_0805_HandSoldering" H 4468 3570 50  0001 C CNN
 F 3 "" H 4430 3720 50  0000 C CNN
 	1    4430 3720
@@
 F 0 "R401" V 4740 3690 50  0000 C CNN
 F 1 "0" V 4660 3690 50  0000 C CNN
-F 2 "" V 4590 3690 50  0000 C CNN
+F 2 "Resistors_SMD:R_0805_HandSoldering" V 4590 3690 50  0001 C CNN
 F 3 "" H 4660 3690 50  0000 C CNN
 	1    4660 3690
@@
 Connection ~ 5280 4060
 Wire Wire Line
-	6150 4060 5830 4060
+	5280 4060 6150 4060
 Wire Wire Line
-	5830 4060 5360 4060
+	6150 4060 6150 3970
 Wire Wire Line
-	5360 4060 5280 4060
-Wire Wire Line
-	6150 3970 6150 4060
-Wire Wire Line
-	5280 4280 5200 4280
-Wire Wire Line
-	5200 4280 5120 4280
-Wire Wire Line
-	5120 4280 4660 4280
-Wire Wire Line
-	4660 4280 4430 4280
+	5280 4280 4430 4280
 Wire Wire Line
 	4430 4280 4430 3870
@@
 	4430 3080 4430 3570
 Wire Wire Line
-	6690 3080 6150 3080
-Wire Wire Line
-	6150 3080 5830 3080
-Wire Wire Line
-	5830 3080 5630 3080
+	5630 3080 6690 3080
 Connection ~ 5280 4280
 Wire Wire Line
-	5280 3640 5280 4060
-Wire Wire Line
-	5280 4060 5280 4280
-Wire Wire Line
-	5280 4280 5280 4310
+	5280 3640 5280 4310
 $Comp
 L LM2931D-R U401
@@
 F 0 "U401" H 5490 3070 50  0000 C CNN
 F 1 "LM2931D-R" H 5240 3630 50  0000 C CNN
-F 2 "" H 5220 3280 50  0000 C CNN
+F 2 "SMD_Packages:SOIC-8-N" H 5220 3280 50  0001 C CNN
 F 3 "" H 5220 3280 50  0000 C CNN
 	1    5220 3280
@@
 F 0 "R402" V 5910 3340 50  0000 C CNN
 F 1 "27K" V 5830 3340 50  0000 C CNN
-F 2 "" V 5760 3340 50  0000 C CNN
+F 2 "Resistors_SMD:R_0805_HandSoldering" V 5760 3340 50  0001 C CNN
 F 3 "" H 5830 3340 50  0000 C CNN
 	1    5830 3340
@@
 F 0 "R403" V 5910 3720 50  0000 C CNN
 F 1 "21.6K" V 5830 3720 50  0000 C CNN
-F 2 "" V 5760 3720 50  0000 C CNN
+F 2 "Resistors_SMD:R_0805_HandSoldering" V 5760 3720 50  0001 C CNN
 F 3 "" H 5830 3720 50  0000 C CNN
 	1    5830 3720
@@
 Connection ~ 5830 3080
 Wire Wire Line
-	5830 3570 5830 3530
-Wire Wire Line
-	5830 3530 5830 3490
+	5830 3490 5830 3570
 Wire Wire Line
 	5830 3870 5830 4060
@@
 Connection ~ 5360 4060
 Wire Wire Line
-	4840 3080 4430 3080
-Wire Wire Line
-	4430 3080 4310 3080
+	4310 3080 4840 3080
 Text HLabel 4310 3080 0    60   Input ~ 0
 Vin

Commit message: Finalizing MPNs and passive values for BOM generation and ordering parts.
Parts:
- C401, C402: value C -> .1; MPN (none) -> 08055C104KAT2A
- U401: MPN (none) -> LM2931D-R
Changed lines of the file:
@@
 Date "2016-06-12"
 Rev "-"
-Comp "J A"
+Comp "Joseph Allan"
 Comment1 ""
 Comment2 ""
@@
 $EndDescr
 $Comp
-L GND #PWR07
+L GND #PWR06
 U 1 1 575DAECE
 P 5280 4310
-F 0 "#PWR07" H 5280 4060 50  0001 C CNN
+F 0 "#PWR06" H 5280 4060 50  0001 C CNN
 F 1 "GND" H 5280 4160 50  0000 C CNN
 F 2 "" H 5280 4310 50  0000 C CNN
@@
 P 6150 3820
 F 0 "C402" H 6175 3920 50  0000 L CNN
-F 1 "C" H 6175 3720 50  0000 L CNN
+F 1 ".1" H 6175 3720 50  0000 L CNN
 F 2 "Capacitors_SMD:C_0805_HandSoldering" H 6188 3670 50  0001 C CNN
 F 3 "" H 6150 3820 50  0000 C CNN
+F 4 "08055C104KAT2A" H 6150 3820 60  0001 C CNN "MPN"
 	1    6150 3820
 	-1   0    0    -1
@@
 P 4430 3720
 F 0 "C401" H 4455 3820 50  0000 L CNN
-F 1 "C" H 4455 3620 50  0000 L CNN
+F 1 ".1" H 4455 3620 50  0000 L CNN
 F 2 "Capacitors_SMD:C_0805_HandSoldering" H 4468 3570 50  0001 C CNN
 F 3 "" H 4430 3720 50  0000 C CNN
+F 4 "08055C104KAT2A" H 4430 3720 60  0001 C CNN "MPN"
 	1    4430 3720
 	-1   0    0    -1
@@
 F 2 "SMD_Packages:SOIC-8-N" H 5220 3280 50  0001 C CNN
 F 3 "" H 5220 3280 50  0000 C CNN
+F 4 "LM2931D-R" H 5220 3280 60  0001 C CNN "MPN"
 	1    5220 3280
 	1    0    0    -1
