File: VoltageControl.sch (KiCad schematic (older format))
At the start: 7 parts

Commit message: Initial annotation.
Parts:
- gave numbers to parts that had none: 7
Changed lines of the file:
@@
 encoding utf-8
 Sheet 3 4
-Title ""
-Date ""
-Rev ""
-Comp ""
+Title "Voltage Control"
+Date "2016-06-12"
+Rev "-"
+Comp "J A"
 Comment1 ""
 Comment2 ""
@@
 $EndDescr
 $Comp
-L LMV358 U?
+L LMV358 U201
 U 2 1 575DE290
 P 5270 3920
-F 0 "U?" H 5220 4120 50  0000 L CNN
+F 0 "U201" H 5220 4120 50  0000 L CNN
 F 1 "LMV358" H 5220 3670 50  0000 L CNN
 F 2 "" H 5270 3920 50  0000 C CNN
@@
 $EndComp
 $Comp
-L R R?
+L R R301
 U 1 1 575DE297
 P 4160 4410
-F 0 "R?" V 4240 4410 50  0000 C CNN
+F 0 "R301" V 4240 4410 50  0000 C CNN
 F 1 "R" V 4160 4410 50  0000 C CNN
 F 2 "" V 4090 4410 50  0000 C CNN
@@
 $EndComp
 $Comp
-L GND #PWR?
+L GND #PWR302
 U 1 1 575DE29E
 P 5170 4330
-F 0 "#PWR?" H 5170 4080 50  0001 C CNN
+F 0 "#PWR302" H 5170 4080 50  0001 C CNN
 F 1 "GND" H 5170 4180 50  0000 C CNN
 F 2 "" H 5170 4330 50  0000 C CNN
@@
 $EndComp
 $Comp
-L POT-RESCUE-CSOS RV?
+L POT-RESCUE-CSOS RV301
 U 1 1 575DE2A4
 P 4160 3790
-F 0 "RV?" H 4160 3690 50  0000 C CNN
+F 0 "RV301" H 4160 3690 50  0000 C CNN
 F 1 "POT" H 4160 3790 50  0000 C CNN
 F 2 "" H 4160 3790 50  0000 C CNN
@@
 	5170 3140 5170 3620
 Wire Wire Line
-	4310 2080 4310 3140
+	4310 2080 4310 3790
 Wire Wire Line
-	4310 3140 4310 3790
-Wire Wire Line
-	4160 5170 6970 5170
-Wire Wire Line
-	6970 5170 7770 5170
+	4160 5170 7770 5170
 Connection ~ 4160 4140
 Wire Wire Line
 	4490 4140 4160 4140
 Wire Wire Line
-	4160 4040 4160 4140
-Wire Wire Line
-	4160 4140 4160 4260
+	4160 4040 4160 4260
 Wire Wire Line
 	4490 3820 4490 4140
@@
 	4740 4550 6970 4550
 $Comp
-L C C?
+L C C301
 U 1 1 575DE2B7
 P 4820 3370
-F 0 "C?" H 4845 3470 50  0000 L CNN
+F 0 "C301" H 4845 3470 50  0000 L CNN
 F 1 "C" H 4845 3270 50  0000 L CNN
 F 2 "" H 4858 3220 50  0000 C CNN
@@
 $EndComp
 $Comp
-L GND #PWR?
+L GND #PWR301
 U 1 1 575DE2BE
 P 4820 3560
-F 0 "#PWR?" H 4820 3310 50  0001 C CNN
+F 0 "#PWR301" H 4820 3310 50  0001 C CNN
 F 1 "GND" H 4820 3410 50  0000 C CNN
 F 2 "" H 4820 3560 50  0000 C CNN
@@
 	4160 4560 4160 5170
 Wire Wire Line
-	4310 3140 4820 3140
-Wire Wire Line
-	4820 3140 5170 3140
+	4310 3140 5170 3140
 Connection ~ 4310 3140
 Wire Wire Line
@@
 2.7V
 $Comp
-L D D?
+L D D301
 U 1 1 575DE840
 P 6010 3920
-F 0 "D?" H 6010 4020 50  0000 C CNN
+F 0 "D301" H 6010 4020 50  0000 C CNN
 F 1 "D" H 6010 3820 50  0000 C CNN
 F 2 "" H 6010 3920 50  0000 C CNN
@@
 $EndComp
 $Comp
-L R R?
+L R R302
 U 1 1 575DE94B
 P 6970 4340
-F 0 "R?" V 7050 4340 50  0000 C CNN
+F 0 "R302" V 7050 4340 50  0000 C CNN
 F 1 "9K" V 6970 4340 50  0000 C CNN
 F 2 "" V 6900 4340 50  0000 C CNN
@@
 $EndComp
 $Comp
-L R R?
+L R R303
 U 1 1 575DEA24
 P 6970 4870
-F 0 "R?" V 7050 4870 50  0000 C CNN
+F 0 "R303" V 7050 4870 50  0000 C CNN
 F 1 "1K" V 6970 4870 50  0000 C CNN
 F 2 "" V 6900 4870 50  0000 C CNN
@@
 $EndComp
 Wire Wire Line
-	6970 4490 6970 4550
-Wire Wire Line
-	6970 4550 6970 4720
+	6970 4490 6970 4720
 Connection ~ 6970 4550
 Wire Wire Line

Commit message: Initial component association and global spread in layout.
Parts:
- C301: footprint (none) -> Capacitors_SMD:C_0805_HandSoldering
- D301: footprint (none) -> Diodes_SMD:SOD-123; MPN (none) -> 1N4148W-7-F
- R301, R302, R303: footprint (none) -> Resistors_SMD:R_0805_HandSoldering
- RV301: footprint (none) -> Potentiometers:Potentiometer_WirePads_largePads
- U201: footprint (none) -> SMD_Packages:SOIC-8-N
Changed lines of the file:
@@
 F 0 "U201" H 5220 4120 50  0000 L CNN
 F 1 "LMV358" H 5220 3670 50  0000 L CNN
-F 2 "" H 5270 3920 50  0000 C CNN
+F 2 "SMD_Packages:SOIC-8-N" H 5270 3920 50  0001 C CNN
 F 3 "" H 5270 3920 50  0000 C CNN
 	2    5270 3920
@@
 F 0 "R301" V 4240 4410 50  0000 C CNN
 F 1 "R" V 4160 4410 50  0000 C CNN
-F 2 "" V 4090 4410 50  0000 C CNN
+F 2 "Resistors_SMD:R_0805_HandSoldering" V 4090 4410 50  0001 C CNN
 F 3 "" H 4160 4410 50  0000 C CNN
 	1    4160 4410
@@
 $EndComp
 $Comp
-L GND #PWR302
+L GND #PWR05
 U 1 1 575DE29E
 P 5170 4330
-F 0 "#PWR302" H 5170 4080 50  0001 C CNN
+F 0 "#PWR05" H 5170 4080 50  0001 C CNN
 F 1 "GND" H 5170 4180 50  0000 C CNN
 F 2 "" H 5170 4330 50  0000 C CNN
@@
 F 0 "RV301" H 4160 3690 50  0000 C CNN
 F 1 "POT" H 4160 3790 50  0000 C CNN
-F 2 "" H 4160 3790 50  0000 C CNN
+F 2 "Potentiometers:Potentiometer_WirePads_largePads" H 4160 3790 50  0001 C CNN
 F 3 "" H 4160 3790 50  0000 C CNN
 	1    4160 3790
@@
 F 0 "C301" H 4845 3470 50  0000 L CNN
 F 1 "C" H 4845 3270 50  0000 L CNN
-F 2 "" H 4858 3220 50  0000 C CNN
+F 2 "Capacitors_SMD:C_0805_HandSoldering" H 4858 3220 50  0001 C CNN
 F 3 "" H 4820 3370 50  0000 C CNN
 	1    4820 3370
@@
 $EndComp
 $Comp
-L GND #PWR301
+L GND #PWR06
 U 1 1 575DE2BE
 P 4820 3560
-F 0 "#PWR301" H 4820 3310 50  0001 C CNN
+F 0 "#PWR06" H 4820 3310 50  0001 C CNN
 F 1 "GND" H 4820 3410 50  0000 C CNN
 F 2 "" H 4820 3560 50  0000 C CNN
@@
 F 0 "D301" H 6010 4020 50  0000 C CNN
 F 1 "D" H 6010 3820 50  0000 C CNN
-F 2 "" H 6010 3920 50  0000 C CNN
-F 3 "" H 6010 3920 50  0000 C CNN
+F 2 "Diodes_SMD:SOD-123" H 6010 3920 50  0001 C CNN
+F 3 "http://www.diodes.com/_files/datasheets/ds30086.pdf" H 6010 3920 50  0001 C CNN
+F 4 "1N4148W-7-F" H 6010 3920 60  0001 C CNN "MPN"
 	1    6010 3920
 	1    0    0    -1
@@
 F 0 "R302" V 7050 4340 50  0000 C CNN
 F 1 "9K" V 6970 4340 50  0000 C CNN
-F 2 "" V 6900 4340 50  0000 C CNN
+F 2 "Resistors_SMD:R_0805_HandSoldering" V 6900 4340 50  0001 C CNN
 F 3 "" H 6970 4340 50  0000 C CNN
 	1    6970 4340
@@
 F 0 "R303" V 7050 4870 50  0000 C CNN
 F 1 "1K" V 6970 4870 50  0000 C CNN
-F 2 "" V 6900 4870 50  0000 C CNN
+F 2 "Resistors_SMD:R_0805_HandSoldering" V 6900 4870 50  0001 C CNN
 F 3 "" H 6970 4870 50  0000 C CNN
 	1    6970 4870

Commit message: Built potentiometer and added to layout.
Parts:
- RV301: footprint Potentiometers:Potentiometer_WirePads_largePads -> CSOS:P090L-02F25BR10K
Changed lines of the file:
@@
 F 0 "RV301" H 4160 3690 50  0000 C CNN
 F 1 "POT" H 4160 3790 50  0000 C CNN
-F 2 "Potentiometers:Potentiometer_WirePads_largePads" H 4160 3790 50  0001 C CNN
+F 2 "CSOS:P090L-02F25BR10K" H 4160 3790 50  0001 C CNN
 F 3 "" H 4160 3790 50  0000 C CNN
 	1    4160 3790

Commit message: Fixing voltage dividers and adding values.
Parts:
- R301: value R -> 28.7K
- RV301: value POT -> 10K
Connections:
- net 2.7V: now also R301.1; no longer RV301.2
- net Current_Sink-: now also RV301.3; no longer R301.2
- new net: R301.2, RV301.2, U201.5 (+)
Other:
- note added: "0-20V"
- note added: "0-2V"
- moved on the sheet: R301, RV301
Changed lines of the file:
@@
 L R R301
 U 1 1 575DE297
-P 4160 4410
-F 0 "R301" V 4240 4410 50  0000 C CNN
-F 1 "R" V 4160 4410 50  0000 C CNN
-F 2 "Resistors_SMD:R_0805_HandSoldering" V 4090 4410 50  0001 C CNN
-F 3 "" H 4160 4410 50  0000 C CNN
-	1    4160 4410
+P 4310 3430
+F 0 "R301" V 4390 3430 50  0000 C CNN
+F 1 "28.7K" V 4310 3430 50  0000 C CNN
+F 2 "Resistors_SMD:R_0805_HandSoldering" V 4240 3430 50  0001 C CNN
+F 3 "" H 4310 3430 50  0000 C CNN
+	1    4310 3430
 	1    0    0    -1
 $EndComp
@@
 L POT-RESCUE-CSOS RV301
 U 1 1 575DE2A4
-P 4160 3790
-F 0 "RV301" H 4160 3690 50  0000 C CNN
-F 1 "POT" H 4160 3790 50  0000 C CNN
-F 2 "CSOS:P090L-02F25BR10K" H 4160 3790 50  0001 C CNN
-F 3 "" H 4160 3790 50  0000 C CNN
-	1    4160 3790
+P 3890 3820
+F 0 "RV301" H 3890 3720 50  0000 C CNN
+F 1 "10K" H 3890 3820 50  0000 C CNN
+F 2 "CSOS:P090L-02F25BR10K" H 3890 3820 50  0001 C CNN
+F 3 "" H 3890 3820 50  0000 C CNN
+	1    3890 3820
 	0    1    1    0
 $EndComp
@@
 	5170 3140 5170 3620
 Wire Wire Line
-	4310 2080 4310 3790
+	4310 2080 4310 3280
 Wire Wire Line
-	4160 5170 7770 5170
-Connection ~ 4160 4140
+	3890 5170 7770 5170
 Wire Wire Line
-	4490 4140 4160 4140
-Wire Wire Line
-	4160 4040 4160 4260
-Wire Wire Line
-	4490 3820 4490 4140
-Wire Wire Line
-	4970 3820 4490 3820
+	4040 3820 4970 3820
 Wire Wire Line
 	5170 4220 5170 4330
@@
 	4820 3560 4820 3520
 Wire Wire Line
-	4160 4560 4160 5170
+	3890 4070 3890 5170
 Wire Wire Line
 	4310 3140 5170 3140
@@
 Text HLabel 7770 5170 2    60   Input ~ 0
 Current_Sink-
+Wire Wire Line
+	4310 3580 4310 3820
+Connection ~ 4310 3820
+Text Notes 4400 3820 0    60   ~ 0
+0-2V
+Text Notes 5790 4550 0    60   ~ 0
+0-2V
+Text Notes 7340 4130 0    60   ~ 0
+0-20V
 $EndSCHEMATC

Commit message: Layout connected.
Parts:
- removed C301: C, Capacitors_SMD:C_0805_HandSoldering, symbol C
Connections:
- net at R301.2, RV301.2: now also U201.3 (+); no longer U201.5 (+)
- net at R302.2, R303.1: now also U201.2 (-); no longer U201.6 (-)
- net at D301.1 (K): now also U201.1; no longer U201.7
Changed lines of the file:
@@
 $Comp
 L LMV358 U201
-U 2 1 575DE290
+U 1 1 575DE290
 P 5270 3920
 F 0 "U201" H 5220 4120 50  0000 L CNN
@@
 F 2 "SMD_Packages:SOIC-8-N" H 5270 3920 50  0001 C CNN
 F 3 "" H 5270 3920 50  0000 C CNN
-	2    5270 3920
+	1    5270 3920
 	1    0    0    -1
 $EndComp
@@
 Wire Wire Line
 	4740 4550 6970 4550
-$Comp
-L C C301
-U 1 1 575DE2B7
-P 4820 3370
-F 0 "C301" H 4845 3470 50  0000 L CNN
-F 1 "C" H 4845 3270 50  0000 L CNN
-F 2 "Capacitors_SMD:C_0805_HandSoldering" H 4858 3220 50  0001 C CNN
-F 3 "" H 4820 3370 50  0000 C CNN
-	1    4820 3370
-	1    0    0    -1
-$EndComp
-$Comp
-L GND #PWR06
-U 1 1 575DE2BE
-P 4820 3560
-F 0 "#PWR06" H 4820 3310 50  0001 C CNN
-F 1 "GND" H 4820 3410 50  0000 C CNN
-F 2 "" H 4820 3560 50  0000 C CNN
-F 3 "" H 4820 3560 50  0000 C CNN
-	1    4820 3560
-	1    0    0    -1
-$EndComp
-Wire Wire Line
-	4820 3560 4820 3520
 Wire Wire Line
 	3890 4070 3890 5170
@@
 Connection ~ 4310 3140
 Wire Wire Line
-	4820 3220 4820 3140
-Connection ~ 4820 3140
-Wire Wire Line
 	5860 3920 5570 3920
